Commit message: rover_gazebo: spawn clear of the Husarion logo, which is 1.8 m tall
The rover was spawning inside solid geometry in this world, invisible in the
viewport and unable to move, while the entity tree, gz model --list and /odom all
showed it present and at the origin.

The logo is not the floor decal it looks like. Every node in husarion_logo.dae
carries a x100 scale matrix. With the world's <scale>6</scale> on top, the logo
is 24.6 x 24.6 m and stands 1.80 m tall, and its 'rectangle' element is a full
plate covering x -11.96..12.66 and y -12.32..12.31. The world origin is inside
it, so the default spawn at z=0.02 put the rover 1.8 m underground. Dropped from
z=2.5 it settles at 1.791, on the roof.

The plate stays at full height: it is the only 3D structure in this world and the
only thing in it worth mapping. What changes is where the rover starts. x:=-13
puts it on open ground a metre off the western edge, where it settles at
z=-0.0006, the same as on flat.sdf. slam_sim.launch.py now passes x, y, z and yaw
through to rover_gazebo, which it did not before, so the spawn can be set from
the top-level launch.

The ground plane goes from Husarion's 25 m to 60 m. Theirs is smaller than the
logo standing on it, so every metre of visible ground was under the plate. A
plane collision is infinite either way, so only the visible square changes.

The world, both READMEs and the pipeline doc previously described this logo as a
0.25 m floor tile sitting off the edge of the plane. That came from measuring the
raw vertex arrays in the mesh and missing the node transforms, and it was wrong
by a factor of 100. All four now carry the measured figures. The world is also
no longer listed as ground-truth-only: a 1.8 m plate is geometry ICP can register
against, so odom_source:=lidar is worth trying here.

Co-Authored-By: Claude Opus 5 <noreply@anthropic.com>
Claude-Session: https://claude.ai/code/session_016UyRUMgQSysnbPBC6fSEvi

File: src/rover_gazebo/urdf/rover.urdf.xacro (robot description, xacro)
@@ -32,4 +32,20 @@
   <xacro:property name="mesh_collision" value="$(arg mesh_collision)"/>
   <!-- ================================================================= -->
+  <!-- Mesh URI.                                                         -->
+  <!--                                                                   -->
+  <!-- Absolute, and deliberately not package://. This model is spawned   -->
+  <!-- from a string, not a file: rover_sim.launch.py runs                -->
+  <!-- 'ros_gz_sim create -topic robot_description'. sdformat rewrites    -->
+  <!-- package:// to model:// and then has no file to resolve it against, -->
+  <!-- so the raw model:// URI reaches the renderer, which silently draws -->
+  <!-- nothing. See doc/GAZEBO_VISUALS.md.                                -->
+  <!--                                                                   -->
+  <!-- An absolute file:// URI needs no resolution at all. xacro expands  -->
+  <!-- $(find rover_gazebo) on the machine that launches, so this stays   -->
+  <!-- correct per machine. resource_retriever reads it, so RViz is       -->
+  <!-- unaffected.                                                       -->
+  <!-- ================================================================= -->
+  <xacro:property name="mesh_uri" value="file://$(find rover_gazebo)/meshes"/>
+  <!-- ================================================================= -->
   <!-- Frame fix.                                                        -->
   <!--                                                                   -->

File: src/rover_gazebo/urdf/rover_body.xacro (robot description, xacro)
@@ -27,5 +27,5 @@
     <visual>
       <origin xyz="0 0 0" rpy="0 0 0"/>
-      <geometry><mesh filename="package://rover_gazebo/meshes/base_link.STL"/></geometry>
+      <geometry><mesh filename="${mesh_uri}/base_link.STL"/></geometry>
       <material name="rover_grey"/>
     </visual>
@@ -46,11 +46,11 @@
     <visual>
       <origin xyz="0 0 0" rpy="0 0 0"/>
-      <geometry><mesh filename="package://rover_gazebo/meshes/FLS.STL"/></geometry>
-      <material name="rover_grey"/>
-    </visual>
-    <xacro:if value="${mesh_collision}">
-      <collision>
-        <origin xyz="0 0 0" rpy="0 0 0"/>
-        <geometry><mesh filename="package://rover_gazebo/meshes/FLS.STL"/></geometry>
+      <geometry><mesh filename="${mesh_uri}/FLS.STL"/></geometry>
+      <material name="rover_grey"/>
+    </visual>
+    <xacro:if value="${mesh_collision}">
+      <collision>
+        <origin xyz="0 0 0" rpy="0 0 0"/>
+        <geometry><mesh filename="${mesh_uri}/FLS.STL"/></geometry>
       </collision>
     </xacro:if>
@@ -66,5 +66,5 @@
     <visual>
       <origin xyz="0 0 0" rpy="0 0 0"/>
-      <geometry><mesh filename="package://rover_gazebo/meshes/LCON.STL"/></geometry>
+      <geometry><mesh filename="${mesh_uri}/LCON.STL"/></geometry>
       <material name="rover_grey"/>
     </visual>
@@ -80,11 +80,11 @@
     <visual>
       <origin xyz="0 0 0" rpy="0 0 0"/>
-      <geometry><mesh filename="package://rover_gazebo/meshes/FLE.STL"/></geometry>
-      <material name="rover_grey"/>
-    </visual>
-    <xacro:if value="${mesh_collision}">
-      <collision>
-        <origin xyz="0 0 0" rpy="0 0 0"/>
-        <geometry><mesh filename="package://rover_gazebo/meshes/FLE.STL"/></geometry>
+      <geometry><mesh filename="${mesh_uri}/FLE.STL"/></geometry>
+      <material name="rover_grey"/>
+    </visual>
+    <xacro:if value="${mesh_collision}">
+      <collision>
+        <origin xyz="0 0 0" rpy="0 0 0"/>
+        <geometry><mesh filename="${mesh_uri}/FLE.STL"/></geometry>
       </collision>
     </xacro:if>
@@ -100,5 +100,5 @@
     <visual>
       <origin xyz="0 0 0" rpy="0 0 0"/>
-      <geometry><mesh filename="package://rover_gazebo/meshes/FLD.STL"/></geometry>
+      <geometry><mesh filename="${mesh_uri}/FLD.STL"/></geometry>
       <material name="rover_grey"/>
     </visual>
@@ -119,11 +119,11 @@
     <visual>
       <origin xyz="0 0 0" rpy="0 0 0"/>
-      <geometry><mesh filename="package://rover_gazebo/meshes/FRS.STL"/></geometry>
-      <material name="rover_grey"/>
-    </visual>
-    <xacro:if value="${mesh_collision}">
-      <collision>
-        <origin xyz="0 0 0" rpy="0 0 0"/>
-        <geometry><mesh filename="package://rover_gazebo/meshes/FRS.STL"/></geometry>
+      <geometry><mesh filename="${mesh_uri}/FRS.STL"/></geometry>
+      <material name="rover_grey"/>
+    </visual>
+    <xacro:if value="${mesh_collision}">
+      <collision>
+        <origin xyz="0 0 0" rpy="0 0 0"/>
+        <geometry><mesh filename="${mesh_uri}/FRS.STL"/></geometry>
       </collision>
     </xacro:if>
@@ -139,5 +139,5 @@
     <visual>
       <origin xyz="0 0 0" rpy="0 0 0"/>
-      <geometry><mesh filename="package://rover_gazebo/meshes/RCON.STL"/></geometry>
+      <geometry><mesh filename="${mesh_uri}/RCON.STL"/></geometry>
       <material name="rover_grey"/>
     </visual>
@@ -153,11 +153,11 @@
     <visual>
       <origin xyz="0 0 0" rpy="0 0 0"/>
-      <geometry><mesh filename="package://rover_gazebo/meshes/FRE.STL"/></geometry>
-      <material name="rover_grey"/>
-    </visual>
-    <xacro:if value="${mesh_collision}">
-      <collision>
-        <origin xyz="0 0 0" rpy="0 0 0"/>
-        <geometry><mesh filename="package://rover_gazebo/meshes/FRE.STL"/></geometry>
+      <geometry><mesh filename="${mesh_uri}/FRE.STL"/></geometry>
+      <material name="rover_grey"/>
+    </visual>
+    <xacro:if value="${mesh_collision}">
+      <collision>
+        <origin xyz="0 0 0" rpy="0 0 0"/>
+        <geometry><mesh filename="${mesh_uri}/FRE.STL"/></geometry>
       </collision>
     </xacro:if>
@@ -173,5 +173,5 @@
     <visual>
       <origin xyz="0 0 0" rpy="0 0 0"/>
-      <geometry><mesh filename="package://rover_gazebo/meshes/FRD.STL"/></geometry>
+      <geometry><mesh filename="${mesh_uri}/FRD.STL"/></geometry>
       <material name="rover_grey"/>
     </visual>
@@ -192,11 +192,11 @@
     <visual>
       <origin xyz="0 0 0" rpy="0 0 0"/>
-      <geometry><mesh filename="package://rover_gazebo/meshes/BRS.STL"/></geometry>
-      <material name="rover_grey"/>
-    </visual>
-    <xacro:if value="${mesh_collision}">
-      <collision>
-        <origin xyz="0 0 0" rpy="0 0 0"/>
-        <geometry><mesh filename="package://rover_gazebo/meshes/BRS.STL"/></geometry>
+      <geometry><mesh filename="${mesh_uri}/BRS.STL"/></geometry>
+      <material name="rover_grey"/>
+    </visual>
+    <xacro:if value="${mesh_collision}">
+      <collision>
+        <origin xyz="0 0 0" rpy="0 0 0"/>
+        <geometry><mesh filename="${mesh_uri}/BRS.STL"/></geometry>
       </collision>
     </xacro:if>
@@ -212,11 +212,11 @@
     <visual>
       <origin xyz="0 0 0" rpy="0 0 0"/>
-      <geometry><mesh filename="package://rover_gazebo/meshes/BRE.STL"/></geometry>
-      <material name="rover_grey"/>
-    </visual>
-    <xacro:if value="${mesh_collision}">
-      <collision>
-        <origin xyz="0 0 0" rpy="0 0 0"/>
-        <geometry><mesh filename="package://rover_gazebo/meshes/BRE.STL"/></geometry>
+      <geometry><mesh filename="${mesh_uri}/BRE.STL"/></geometry>
+      <material name="rover_grey"/>
+    </visual>
+    <xacro:if value="${mesh_collision}">
+      <collision>
+        <origin xyz="0 0 0" rpy="0 0 0"/>
+        <geometry><mesh filename="${mesh_uri}/BRE.STL"/></geometry>
       </collision>
     </xacro:if>
@@ -232,5 +232,5 @@
     <visual>
       <origin xyz="0 0 0" rpy="0 0 0"/>
-      <geometry><mesh filename="package://rover_gazebo/meshes/BRD.STL"/></geometry>
+      <geometry><mesh filename="${mesh_uri}/BRD.STL"/></geometry>
       <material name="rover_grey"/>
     </visual>
@@ -251,5 +251,5 @@
     <visual>
       <origin xyz="0 0 0" rpy="0 0 0"/>
-      <geometry><mesh filename="package://rover_gazebo/meshes/Rdiffcon2.STL"/></geometry>
+      <geometry><mesh filename="${mesh_uri}/Rdiffcon2.STL"/></geometry>
       <material name="rover_grey"/>
     </visual>
@@ -265,11 +265,11 @@
     <visual>
       <origin xyz="0 0 0" rpy="0 0 0"/>
-      <geometry><mesh filename="package://rover_gazebo/meshes/BLS.STL"/></geometry>
-      <material name="rover_grey"/>
-    </visual>
-    <xacro:if value="${mesh_collision}">
-      <collision>
-        <origin xyz="0 0 0" rpy="0 0 0"/>
-        <geometry><mesh filename="package://rover_gazebo/meshes/BLS.STL"/></geometry>
+      <geometry><mesh filename="${mesh_uri}/BLS.STL"/></geometry>
+      <material name="rover_grey"/>
+    </visual>
+    <xacro:if value="${mesh_collision}">
+      <collision>
+        <origin xyz="0 0 0" rpy="0 0 0"/>
+        <geometry><mesh filename="${mesh_uri}/BLS.STL"/></geometry>
       </collision>
     </xacro:if>
@@ -285,11 +285,11 @@
     <visual>
       <origin xyz="0 0 0" rpy="0 0 0"/>
-      <geometry><mesh filename="package://rover_gazebo/meshes/BLE.STL"/></geometry>
-      <material name="rover_grey"/>
-    </visual>
-    <xacro:if value="${mesh_collision}">
-      <collision>
-        <origin xyz="0 0 0" rpy="0 0 0"/>
-        <geometry><mesh filename="package://rover_gazebo/meshes/BLE.STL"/></geometry>
+      <geometry><mesh filename="${mesh_uri}/BLE.STL"/></geometry>
+      <material name="rover_grey"/>
+    </visual>
+    <xacro:if value="${mesh_collision}">
+      <collision>
+        <origin xyz="0 0 0" rpy="0 0 0"/>
+        <geometry><mesh filename="${mesh_uri}/BLE.STL"/></geometry>
       </collision>
     </xacro:if>
@@ -305,5 +305,5 @@
     <visual>
       <origin xyz="0 0 0" rpy="0 0 0"/>
-      <geometry><mesh filename="package://rover_gazebo/meshes/BLD.STL"/></geometry>
+      <geometry><mesh filename="${mesh_uri}/BLD.STL"/></geometry>
       <material name="rover_grey"/>
     </visual>
@@ -324,5 +324,5 @@
     <visual>
       <origin xyz="0 0 0" rpy="0 0 0"/>
-      <geometry><mesh filename="package://rover_gazebo/meshes/Ldiffcon2.STL"/></geometry>
+      <geometry><mesh filename="${mesh_uri}/Ldiffcon2.STL"/></geometry>
       <material name="rover_grey"/>
     </visual>
@@ -338,5 +338,5 @@
     <visual>
       <origin xyz="0 0 0" rpy="0 0 0"/>
-      <geometry><mesh filename="package://rover_gazebo/meshes/Differential.STL"/></geometry>
+      <geometry><mesh filename="${mesh_uri}/Differential.STL"/></geometry>
       <material name="rover_grey"/>
     </visual>
@@ -352,5 +352,5 @@
     <visual>
       <origin xyz="0 0 0" rpy="0 0 0"/>
-      <geometry><mesh filename="package://rover_gazebo/meshes/Ldiff.STL"/></geometry>
+      <geometry><mesh filename="${mesh_uri}/Ldiff.STL"/></geometry>
       <material name="rover_grey"/>
     </visual>
@@ -366,5 +366,5 @@
     <visual>
       <origin xyz="0 0 0" rpy="0 0 0"/>
-      <geometry><mesh filename="package://rover_gazebo/meshes/Ldiffcon.STL"/></geometry>
+      <geometry><mesh filename="${mesh_uri}/Ldiffcon.STL"/></geometry>
       <material name="rover_grey"/>
     </visual>
@@ -380,5 +380,5 @@
     <visual>
       <origin xyz="0 0 0" rpy="0 0 0"/>
-      <geometry><mesh filename="package://rover_gazebo/meshes/Rdiff.STL"/></geometry>
+      <geometry><mesh filename="${mesh_uri}/Rdiff.STL"/></geometry>
       <material name="rover_grey"/>
     </visual>
@@ -394,5 +394,5 @@
     <visual>
       <origin xyz="0 0 0" rpy="0 0 0"/>
-      <geometry><mesh filename="package://rover_gazebo/meshes/Rdiffcon.STL"/></geometry>
+      <geometry><mesh filename="${mesh_uri}/Rdiffcon.STL"/></geometry>
       <material name="rover_grey"/>
     </visual>

File: src/rover_gazebo/urdf/rover_gazebo.xacro (robot description, xacro)
@@ -33,5 +33,4 @@
       <minDepth>0.001</minDepth>
       <maxVel>0.1</maxVel>
-      <material>Gazebo/DarkGrey</material>
     </gazebo>
   </xacro:macro>
@@ -40,8 +39,11 @@
   <xacro:wheel_contact name="BLD"/>
   <xacro:wheel_contact name="BRD"/>
+  <!-- No <material> here or in wheel_contact. sdformat turns a Gazebo-Classic
+       material name into a <script> pointing at gazebo.material, an Ogre script
+       Harmonic cannot read, and it overrides the RGBA the URDF already carries.
+       Colour is set once, in rover_body.xacro's rover_grey. -->
   <gazebo reference="chassis_link">
     <mu1>0.5</mu1>
     <mu2>0.5</mu2>
-    <material>Gazebo/Grey</material>
   </gazebo>
   <!-- The connector bars and the differential chain overlap their neighbours by
