Commit message: added_teleop_gui_explicit_modes_and_fixed_ackermann_bugs

File: src/rover_gazebo/urdf/rover.urdf.xacro (robot description, xacro)
@@ -6,9 +6,11 @@
     1. The suspension contains four closed kinematic loops. URDF is a tree, so the
        loops cannot be written down and the suspension falls apart without them.
-       Fixed in rover_body.xacro: the loop-closing joints get effort interfaces and
-       are held together at runtime by rocker_coupling_node, which applies the
-       constraints as torques. Gazebo has no solver-level way to enforce them
-       (no <mimic> support), so this is the only coupling mechanism this package
-       ships.
+       Fixed in rover_body.xacro: by default (suspension:=torque) the loop-closing
+       joints get effort interfaces and are held together at runtime by
+       rocker_coupling_node, which applies the constraints as torques, since DART
+       (the default engine) has no solver-level way to enforce them (no <mimic>
+       support). suspension:=mimic uses real <mimic> joints instead, enforced by the
+       physics solver itself; Bullet-Featherstone only, see the suspension argument
+       below and doc/VERIFICATION.md.
     2. The export is Y-up. Spawned as-is the rover lies on its side.
        Fixed below, by a rotated fixed joint under a ROS-convention base_link.
@@ -21,4 +23,12 @@
                                 chassis, rockers and knuckles.
     ros2_control    true        false strips the hardware interface, for RViz-only use.
+    suspension      torque      'torque': the four rockers are held by
+                                rocker_coupling_node's virtual constraint torques (see
+                                rover_body.xacro/rover_ros2_control.xacro); works on
+                                every engine, including DART, the default. 'mimic':
+                                BLS/BRS/FRS are held by real <mimic> joints instead and
+                                FLS by rocker_hold_node.py; Bullet-Featherstone only,
+                                since DART silently ignores <mimic> and would leave
+                                the suspension uncontrolled; see doc/VERIFICATION.md.
 -->
 <robot name="rover" xmlns:xacro="http://www.ros.org/wiki/xacro">
@@ -28,7 +38,9 @@
   <xacro:arg name="ros2_control"   default="true"/>
   <xacro:arg name="controllers_file" default="$(find rover_gazebo)/config/controllers.yaml"/>
+  <xacro:arg name="suspension"     default="torque"/>
   <xacro:property name="sim"            value="$(arg sim)"/>
   <xacro:property name="mass_scale"     value="$(arg mass_scale)"/>
   <xacro:property name="mesh_collision" value="$(arg mesh_collision)"/>
+  <xacro:property name="suspension"     value="$(arg suspension)"/>
   <!-- ================================================================= -->
   <!-- Frame fix.                                                        -->

File: src/rover_gazebo/urdf/rover_body.xacro (robot description, xacro)
@@ -440,4 +440,12 @@
       <limit lower="-0.6" upper="0.6" effort="5000.0" velocity="20.0"/>
       <dynamics damping="5.0" friction="0.5"/>
+      <!-- suspension:=mimic only (rover.urdf.xacro); Bullet-Featherstone, DART
+           ignores this tag entirely; see rocker_hold_node.py. Ratio from
+           config/rover_kinematics.yaml's coupling.followers, chained onto
+           FLS_joint by tools/generate_description.py so it stays correct across
+           a CAD regeneration. -->
+      <xacro:if value="${suspension == 'mimic'}">
+        <mimic joint="FLS_joint" multiplier="-1.007737" offset="0.0"/>
+      </xacro:if>
   </joint>
   <!-- decorative; fixed so sdformat folds it into its parent. Nothing
@@ -474,4 +482,8 @@
       <limit lower="-0.6" upper="0.6" effort="5000.0" velocity="20.0"/>
       <dynamics damping="5.0" friction="0.5"/>
+      <!-- suspension:=mimic only; see FRS_joint's mimic above. -->
+      <xacro:if value="${suspension == 'mimic'}">
+        <mimic joint="FLS_joint" multiplier="0.577165" offset="0.0"/>
+      </xacro:if>
   </joint>
   <joint name="BRE_joint" type="revolute">
@@ -506,4 +518,8 @@
       <limit lower="-0.6" upper="0.6" effort="5000.0" velocity="20.0"/>
       <dynamics damping="5.0" friction="0.5"/>
+      <!-- suspension:=mimic only; see FRS_joint's mimic above. -->
+      <xacro:if value="${suspension == 'mimic'}">
+        <mimic joint="FLS_joint" multiplier="-0.577165" offset="0.0"/>
+      </xacro:if>
   </joint>
   <joint name="BLE_joint" type="revolute">

File: src/rover_gazebo/urdf/rover_ros2_control.xacro (robot description, xacro)
@@ -3,8 +3,23 @@
   ros2_control interfaces.
   Eight driven joints: four steering knuckles under position control and four wheels
-  under velocity control. All four rockers, the free suspension joint and its three
-  dependent followers, get effort interfaces: rocker_coupling_node applies the
-  suspension's closed-loop constraints through them, since Gazebo has no
-  solver-level way to enforce those constraints itself.
+  under velocity control. Both also carry an effort command interface, unused by
+  steer_controller/wheel_controller but claimed by steer_pid_controller/
+  wheel_pid_controller (see controllers.yaml) when explicit_pid mode (control_node.py)
+  is active. Only one of the two controllers on a joint is ever *active* at a time,
+  since rover_kinematics_node switches between them via the controller_manager, so
+  this is never two control laws actually fighting over the joint, just two possible
+  ones. The effort limits below are a hard backstop, not a tuned value: control_node.py's
+  own steer_max_effort/wheel_max_effort parameters (config/rover_control.yaml) are
+  the meaningful, software-side clamp and are set noticeably tighter than these.
+  The rockers depend on the suspension arg (rover.urdf.xacro). suspension:=torque
+  (default, every engine including DART): all four get an effort interface, and
+  rocker_coupling_node applies the suspension's closed-loop constraints through them
+  every cycle, since Gazebo has no solver-level way to enforce those constraints
+  itself. suspension:=mimic (Bullet-Featherstone only): BLS/BRS/FRS get no command
+  interface at all; they're held by real <mimic> joints instead
+  (rover_body.xacro), physics-solver-enforced, and only FLS_joint, the mechanism's
+  one genuinely free coordinate, keeps an effort interface, held by
+  rocker_hold_node.py's single-joint hold. See doc/VERIFICATION.md for why DART
+  can't take the mimic path at all.
 -->
 <robot xmlns:xacro="http://www.ros.org/wiki/xacro">
@@ -16,4 +31,10 @@
         <param name="min">-1.75</param>
         <param name="max">1.75</param>
+      </command_interface>
+      <!-- Backstop only; see the file header. Unmeasured: nothing about this
+           knuckle's real inertia or friction has been characterised yet. -->
+      <command_interface name="effort">
+        <param name="min">-150.0</param>
+        <param name="max">150.0</param>
       </command_interface>
       <state_interface name="position"/>
@@ -27,4 +48,9 @@
         <param name="min">-30.0</param>
         <param name="max">30.0</param>
+      </command_interface>
+      <!-- Backstop only; see the file header. Unmeasured, same as the steer joints'. -->
+      <command_interface name="effort">
+        <param name="min">-150.0</param>
+        <param name="max">150.0</param>
       </command_interface>
       <state_interface name="position"/>
@@ -45,8 +71,4 @@
     <xacro:drive_joint name="BLD_joint"/>
     <xacro:drive_joint name="BRD_joint"/>
-    <!-- Suspension. All four rockers become torque-driven, because a constraint has
-         to push on both joints it ties together. Holding only the followers would
-         let the rear wheels carry load the front rockers never feel, which is not
-         the mechanism the CAD describes. -->
     <xacro:macro name="coupled_rocker" params="name">
       <joint name="${name}">
@@ -60,8 +82,23 @@
       </joint>
     </xacro:macro>
-    <xacro:coupled_rocker name="FLS_joint"/>
-    <xacro:coupled_rocker name="BLS_joint"/>
-    <xacro:coupled_rocker name="BRS_joint"/>
-    <xacro:coupled_rocker name="FRS_joint"/>
+    <xacro:macro name="mimic_follower" params="name">
+      <joint name="${name}">
+        <state_interface name="position"/>
+        <state_interface name="velocity"/>
+        <state_interface name="effort"/>
+      </joint>
+    </xacro:macro>
+    <xacro:if value="${suspension == 'mimic'}">
+      <xacro:coupled_rocker name="FLS_joint"/>
+      <xacro:mimic_follower name="BLS_joint"/>
+      <xacro:mimic_follower name="BRS_joint"/>
+      <xacro:mimic_follower name="FRS_joint"/>
+    </xacro:if>
+    <xacro:unless value="${suspension == 'mimic'}">
+      <xacro:coupled_rocker name="FLS_joint"/>
+      <xacro:coupled_rocker name="BLS_joint"/>
+      <xacro:coupled_rocker name="BRS_joint"/>
+      <xacro:coupled_rocker name="FRS_joint"/>
+    </xacro:unless>
   </ros2_control>
 </robot>

Commit message: implemented the pid and integrated wiith whole pipeline

File: src/rover_gazebo/urdf/rover.urdf.xacro (robot description, xacro)
@@ -6,9 +6,11 @@
     1. The suspension contains four closed kinematic loops. URDF is a tree, so the
        loops cannot be written down and the suspension falls apart without them.
-       Fixed in rover_body.xacro: the loop-closing joints get effort interfaces and
-       are held together at runtime by rocker_coupling_node, which applies the
-       constraints as torques. Gazebo has no solver-level way to enforce them
-       (no <mimic> support), so this is the only coupling mechanism this package
-       ships.
+       Fixed in rover_body.xacro: by default (suspension:=torque) the loop-closing
+       joints get effort interfaces and are held together at runtime by
+       rocker_coupling_node, which applies the constraints as torques, since DART
+       (the default engine) has no solver-level way to enforce them (no <mimic>
+       support). suspension:=mimic uses real <mimic> joints instead, enforced by the
+       physics solver itself; Bullet-Featherstone only, see the suspension argument
+       below and doc/VERIFICATION.md.
     2. The export is Y-up. Spawned as-is the rover lies on its side.
        Fixed below, by a rotated fixed joint under a ROS-convention base_link.
@@ -21,4 +23,12 @@
                                 chassis, rockers and knuckles.
     ros2_control    true        false strips the hardware interface, for RViz-only use.
+    suspension      torque      'torque': the four rockers are held by
+                                rocker_coupling_node's virtual constraint torques (see
+                                rover_body.xacro/rover_ros2_control.xacro); works on
+                                every engine, including DART, the default. 'mimic':
+                                BLS/BRS/FRS are held by real <mimic> joints instead and
+                                FLS by rocker_hold_node.py; Bullet-Featherstone only,
+                                since DART silently ignores <mimic> and would leave
+                                the suspension uncontrolled; see doc/VERIFICATION.md.
 -->
 <robot name="rover" xmlns:xacro="http://www.ros.org/wiki/xacro">
@@ -28,7 +38,9 @@
   <xacro:arg name="ros2_control"   default="true"/>
   <xacro:arg name="controllers_file" default="$(find rover_gazebo)/config/controllers.yaml"/>
+  <xacro:arg name="suspension"     default="torque"/>
   <xacro:property name="sim"            value="$(arg sim)"/>
   <xacro:property name="mass_scale"     value="$(arg mass_scale)"/>
   <xacro:property name="mesh_collision" value="$(arg mesh_collision)"/>
+  <xacro:property name="suspension"     value="$(arg suspension)"/>
   <!-- ================================================================= -->
   <!-- Mesh URI.                                                         -->

File: src/rover_gazebo/urdf/rover_body.xacro (robot description, xacro)
@@ -440,4 +440,12 @@
       <limit lower="-0.6" upper="0.6" effort="5000.0" velocity="20.0"/>
       <dynamics damping="5.0" friction="0.5"/>
+      <!-- suspension:=mimic only (rover.urdf.xacro); Bullet-Featherstone, DART
+           ignores this tag entirely; see rocker_hold_node.py. Ratio from
+           config/rover_kinematics.yaml's coupling.followers, chained onto
+           FLS_joint by tools/generate_description.py so it stays correct across
+           a CAD regeneration. -->
+      <xacro:if value="${suspension == 'mimic'}">
+        <mimic joint="FLS_joint" multiplier="-1.007737" offset="0.0"/>
+      </xacro:if>
   </joint>
   <!-- decorative; fixed so sdformat folds it into its parent. Nothing
@@ -474,4 +482,8 @@
       <limit lower="-0.6" upper="0.6" effort="5000.0" velocity="20.0"/>
       <dynamics damping="5.0" friction="0.5"/>
+      <!-- suspension:=mimic only; see FRS_joint's mimic above. -->
+      <xacro:if value="${suspension == 'mimic'}">
+        <mimic joint="FLS_joint" multiplier="0.577165" offset="0.0"/>
+      </xacro:if>
   </joint>
   <joint name="BRE_joint" type="revolute">
@@ -506,4 +518,8 @@
       <limit lower="-0.6" upper="0.6" effort="5000.0" velocity="20.0"/>
       <dynamics damping="5.0" friction="0.5"/>
+      <!-- suspension:=mimic only; see FRS_joint's mimic above. -->
+      <xacro:if value="${suspension == 'mimic'}">
+        <mimic joint="FLS_joint" multiplier="-0.577165" offset="0.0"/>
+      </xacro:if>
   </joint>
   <joint name="BLE_joint" type="revolute">
