Commit message: feat(rover_gazebo, rover_ekf): add a simulated GPS sensor and wheel-slip residual covariance
Adds a navsat-type GPS sensor to the rover (rover_sensors.xacro), the
world-level NavSat system plugin and spherical_coordinates origin it needs
(empty_world.sdf), and its gz->ROS bridge entry (bridge.yaml). Currently
zero-noise (ideal): Gazebo's navsat sensor applies its noise stddev directly
to lat/lon degrees rather than metres as the schema docs claim, which first
surfaced as wild EKF jumps even at rest -- documented in the xacro's comment
for whenever real noise goes back in. covariance_relay.py relays the bridged
/gps/raw (which carries no covariance at all) to /gps/fix with a small
placeholder covariance, the same pattern it already used for odom/imu.

wheel_body_velocity.py's rigid-body least-squares fit now also tracks its own
residual and folds it into the published yaw-rate covariance, so the EKF
automatically distrusts the wheels when they disagree with each other (e.g.
asymmetric wall contact) instead of trusting a fixed, slip-blind variance.
This can't catch slip that moves every wheel by the same wrong amount (a
flush head-on collision); that case needs a motion source outside the wheels
entirely, which is what the GPS path above is for.

ekf_rover_gazebo.launch.py passes the new gps_topic through to
covariance_relay and defaults use_imu to true. ekf_rover_gazebo_imu.yaml now
also fuses linear acceleration (with gravity removed).

Co-Authored-By: Claude Sonnet 5 <noreply@anthropic.com>

File: src/rover_gazebo/urdf/rover_sensors.xacro (robot description, xacro)
@@ -10,6 +10,11 @@
     camera_link     RGBD camera, front mount, /camera at 15 Hz, plus the
                     REP-103 optical frame the image data is published in
-  The gpu lidar and RGBD camera need the Sensors system (ogre2) and the IMU
-  needs the Imu system in the world; the shipped worlds load both. Topics are
+    gps_link        GPS/GNSS, roof mount, /gps/raw at 5 Hz (NavSatFix, no
+                    covariance: rover_ekf's covariance_relay fills that in
+                    on /gps/fix)
+  The gpu lidar and RGBD camera need the Sensors system (ogre2), the IMU needs
+  the Imu system, and the GPS needs the NavSat system, all in the world; the
+  shipped worlds load them. The world also needs a <spherical_coordinates>
+  origin or the GPS sensor has nothing to measure lat/lon against. Topics are
   bridged in config/bridge.yaml.
 -->
@@ -150,3 +155,44 @@
     </sensor>
   </gazebo>
+  <link name="gps_link">
+    <inertial>
+      <origin xyz="0 0 0" rpy="0 0 0"/>
+      <mass value="0.02"/>
+      <inertia ixx="1e-06" ixy="0" ixz="0" iyy="1e-06" iyz="0" izz="1e-06"/>
+    </inertial>
+    <visual>
+      <origin xyz="0 0 0" rpy="0 0 0"/>
+      <geometry><cylinder radius="0.015" length="0.01"/></geometry>
+      <material name="gps_white"><color rgba="0.9 0.9 0.9 1"/></material>
+    </visual>
+  </link>
+  <joint name="gps_joint" type="fixed">
+    <origin xyz="0 0.2 0.05" rpy="${ros_frame}"/>
+    <parent link="chassis_link"/>
+    <child link="gps_link"/>
+  </joint>
+  <gazebo reference="gps_link">
+    <sensor name="gps_sensor" type="navsat">
+      <always_on>1</always_on>
+      <update_rate>5</update_rate>
+      <topic>/gps/raw</topic>
+      <gz_frame_id>gps_link</gz_frame_id>
+      <navsat>
+        <!-- Ideal for now: zero noise. position_sensing's noise is applied
+             directly to lat/lon in degrees, not converted from the metres the
+             schema docs describe (checked empirically: a stddev of 1.5 here
+             scattered readings across several degrees, i.e. hundreds of km).
+             Keep that in mind if real noise goes back in: deg-equivalents of
+             metres are tiny (1 deg latitude is ~111320 m). -->
+        <position_sensing>
+          <horizontal><noise type="gaussian"><mean>0.0</mean><stddev>0.0</stddev></noise></horizontal>
+          <vertical><noise type="gaussian"><mean>0.0</mean><stddev>0.0</stddev></noise></vertical>
+        </position_sensing>
+        <velocity_sensing>
+          <horizontal><noise type="gaussian"><mean>0.0</mean><stddev>0.0</stddev></noise></horizontal>
+          <vertical><noise type="gaussian"><mean>0.0</mean><stddev>0.0</stddev></noise></vertical>
+        </velocity_sensing>
+      </navsat>
+    </sensor>
+  </gazebo>
 </robot>
